File: ecad/template.kicad_pcb (KiCad board)
At the start: 2 copper layers, 25.2 x 27.3 mm, 3 parts, among them P1 CF_EXP_LEFT, P2 CF_EXP_RIGHT

Commit message: Convert to KiCad 9.0
Other:
- net class Default removed
