File: ecad/template.kicad_pcb (KiCad board)
At the start: 2 copper layers, 25.2 x 27.3 mm, 3 parts, among them P1 CF_EXP_LEFT, P2 CF_EXP_RIGHT

Commit message: Footprints working
Parts:
- removed P1: CF_EXP_LEFT, connectors:BF090-10-X-B2
- removed P2: CF_EXP_RIGHT, connectors:BF090-10-X-B2
- added J1: Conn_01x03, Connector_PinHeader_2.54mm:PinHeader_1x03_P2.54mm_Horizontal, F.Cu at (40.1, 75.0)
- added J2: Conn_01x03, Connector_PinHeader_2.54mm:PinHeader_1x03_P2.54mm_Horizontal, F.Cu at (40.1, 84.7)
- added J3: Conn_01x03, Connector_PinHeader_2.54mm:PinHeader_1x03_P2.54mm_Horizontal, F.Cu at (40.1, 94.4)
- added J4: Conn_01x03, Connector_PinHeader_2.54mm:PinHeader_1x03_P2.54mm_Horizontal, F.Cu at (40.1, 104.1)
- added J5: Conn_01x03, Connector_PinHeader_2.54mm:PinHeader_1x03_P2.54mm_Horizontal, F.Cu at (40.1, 113.8)
- added J6: Conn_01x03, Connector_PinHeader_2.54mm:PinHeader_1x03_P2.54mm_Horizontal, F.Cu at (40.1, 123.5)
- added J7: Conn_01x01, Crazyflie:Servo_Power_GND_2.0x1.5mm, F.Cu at (135.5, 93.0)
- added J8: Conn_01x01, Crazyflie:Servo_Power_GND_2.0x1.5mm, F.Cu at (134.5, 100.5)
- added J9: Conn_02x10_Counter_Clockwise, Crazyflie:Crazyflie_DeckHeader_2x10_P2.00_Vertical, F.Cu at (139.0, 97.0)
- added R1: 500k, Resistor_SMD:R_0603_1608Metric_Pad0.98x0.95mm_HandSolder, F.Cu at (146.0, 98.0)
- added R2: 100k, Resistor_SMD:R_0603_1608Metric_Pad0.98x0.95mm_HandSolder, F.Cu at (146.1, 101.5)

Commit message: Routing
Parts:
- moved J6 108.4 mm to (148.0, 113.1), turned to -90 degrees
- moved J1 103.0 mm to (143.0, 80.9), turned to 90 degrees
- moved J5 94.9 mm to (135.0, 113.1), turned to -90 degrees
- moved J2 89.9 mm to (130.0, 80.9), turned to 90 degrees
- moved J4 84.9 mm to (125.0, 106.0), turned to 180 degrees
- moved J3 84.9 mm to (125.0, 93.1), turned to 180 degrees
- moved J8 14.0 mm to (148.5, 101.5), turned to 90 degrees
- moved J7 13.0 mm to (148.5, 92.5), turned to -90 degrees
- moved R2 7.62 mm to (139.1, 98.5)
- moved R1 7.35 mm to (139.1, 95.5), turned to 180 degrees
Routing:
- net /PWM2: track 0.00 -> 52.8 mm
- net /PWM1: track 0.00 -> 47.1 mm
- net /PWM6: track 0.00 -> 34.3 mm
- net /PWM5: track 0.00 -> 33.3 mm
- net /PWM3: track 0.00 -> 28.2 mm
- net /PWM4: track 0.00 -> 27.5 mm
- net /VBAT_MONITOR: track 0.00 -> 16.0 mm
- net GND: track 0.00 -> 9.71 mm
- net +BATT: track 0.00 -> 7.91 mm
- added copper zone on In1.Cu, net +BATT
- added copper zone on In2.Cu, net +BATT
- added copper zone on In1.Cu, net GND
Other:
- board size 25.2 x 27.3 mm -> 31 x 41 mm
- copper layers 2 -> 4

Commit message: Logan's changes
Parts:
- added C1: 10u, Capacitor_SMD:C_0805_2012Metric_Pad1.18x1.45mm_HandSolder, B.Cu at (131.3, 115.8)
- added C2: 10u, Capacitor_SMD:C_0805_2012Metric_Pad1.18x1.45mm_HandSolder, B.Cu at (144.3, 115.8)
- added C3: 10u, Capacitor_SMD:C_0805_2012Metric_Pad1.18x1.45mm_HandSolder, B.Cu at (155.8, 104.8)
- added C4: 10u, Capacitor_SMD:C_0805_2012Metric_Pad1.18x1.45mm_HandSolder, B.Cu at (155.8, 91.8)
- added C5: 10u, Capacitor_SMD:C_0805_2012Metric_Pad1.18x1.45mm_HandSolder, B.Cu at (146.8, 78.3)
- added C6: 10u, Capacitor_SMD:C_0805_2012Metric_Pad1.18x1.45mm_HandSolder, B.Cu at (133.8, 78.3)
- R1: value 500k -> 200k; footprint Resistor_SMD:R_0603_1608Metric_Pad0.98x0.95mm_HandSolder -> Resistor_SMD:R_0805_2012Metric_Pad1.20x1.40mm_HandSolder
- R2: footprint Resistor_SMD:R_0603_1608Metric_Pad0.98x0.95mm_HandSolder -> Resistor_SMD:R_0805_2012Metric_Pad1.20x1.40mm_HandSolder
- moved J2 37.0 mm to (148.0, 113.1), turned to -90 degrees
- moved J6 37.0 mm to (130.0, 80.9), turned to 90 degrees
- moved J4 33.4 mm to (153.1, 88.0), turned to 0 degrees
- moved J1 33.2 mm to (135.0, 113.1), turned to -90 degrees
- moved J5 33.2 mm to (143.0, 80.9), turned to 90 degrees
- moved J3 29.2 mm to (153.1, 100.9), turned to 0 degrees
- moved J7 19.2 mm to (129.3, 92.5)
- moved J8 19.2 mm to (129.3, 101.5)
- moved R2 0.50 mm to (139.1, 99.0), turned to 180 degrees
- moved R1 0.25 mm to (139.1, 95.3), turned to 0 degrees
Routing:
- net /PWM2: track 52.8 -> 11.2 mm
- net /PWM1: track 47.1 -> 8.15 mm
- net /PWM6: track 34.3 -> 11.9 mm
- net +BATT: track 7.91 -> 26.3 mm
- net GND: track 9.71 -> 28.0 mm
- net /PWM5: track 33.3 -> 16.2 mm
- net /PWM3: track 28.2 -> 14.9 mm
- net /PWM4: track 27.5 -> 23.7 mm
- net /VBAT_MONITOR: track 16.0 -> 17.3 mm
- added copper zone on In2.Cu, net GND
- removed copper zone on In2.Cu, net +BATT
- removed copper zone on In1.Cu, net GND
Other:
- outline, holes or cut-outs redrawn
